File: Power.kicad_sch (KiCad schematic)
At the start: 39 parts, among them U2 SCT2420, U3 SCT2610

Commit message: 优化电源布局,优化中
Changed lines of the file:
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@@
 	(text "DC/DC \n24V转12V"
 		(exclude_from_sim no)
-		(at 91.694 25.654 0)
+		(at 55.118 19.812 0)
 		(effects
 			(font
@@
 	)
 	(table
-		(column_count 2)
+		(column_count 3)
 		(border
 			(external yes)
@@
 			)
 		)
-		(column_widths 10.16 10.16)
-		(row_heights 2.54 2.54 2.54 2.54 2.54)
+		(column_widths 7.62 8.89 8.89)
+		(row_heights 2.54 2.54 2.54 2.54)
 		(cells
-			(table_cell "Fsw"
+			(table_cell "Vout"
 				(exclude_from_sim no)
-				(at 220.98 128.27 0)
-				(size 10.16 2.54)
+				(at 215.9 142.24 0)
+				(size 7.62 2.54)
 				(margins 0.9525 0.9525 0.9525 0.9525)
 				(span 1 1)
@@
 				)
 			)
-			(table_cell "R"
+			(table_cell "R_上"
 				(exclude_from_sim no)
-				(at 231.14 128.27 0)
-				(size 10.16 2.54)
+				(at 223.52 142.24 0)
+				(size 8.89 2.54)
 				(margins 0.9525 0.9525 0.9525 0.9525)
 				(span 1 1)
@@
 				)
 			)
-			(table_cell "200KHz"
+			(table_cell "R_下"
 				(exclude_from_sim no)
-				(at 220.98 130.81 0)
-				(size 10.16 2.54)
+				(at 232.41 142.24 0)
+				(size 8.89 2.54)
 				(margins 0.9525 0.9525 0.9525 0.9525)
 				(span 1 1)
@@
 				)
 			)
-			(table_cell "500K"
+			(table_cell "3.3V"
 				(exclude_from_sim no)
-				(at 231.14 130.81 0)
-				(size 10.16 2.54)
+				(at 215.9 144.78 0)
+				(size 7.62 2.54)
 				(margins 0.9525 0.9525 0.9525 0.9525)
 				(span 1 1)
@@
 				)
 			)
-			(table_cell "330KHz"
+			(table_cell "31.6K"
 				(exclude_from_sim no)
-				(at 220.98 133.35 0)
-				(size 10.16 2.54)
+				(at 223.52 144.78 0)
+				(size 8.89 2.54)
 				(margins 0.9525 0.9525 0.9525 0.9525)
 				(span 1 1)
@@
 				)
 			)
-			(table_cell "301K"
+			(table_cell "10.2K"
 				(exclude_from_sim no)
-				(at 231.14 133.35 0)
-				(size 10.16 2.54)
+				(at 232.41 144.78 0)
+				(size 8.89 2.54)
 				(margins 0.9525 0.9525 0.9525 0.9525)
 				(span 1 1)
@@
 				)
 			)
-			(table_cell "500KHz"
+			(table_cell "12V"
 				(exclude_from_sim no)
-				(at 220.98 135.89 0)
-				(size 10.16 2.54)
+				(at 215.9 147.32 0)
+				(size 7.62 2.54)
 				(margins 0.9525 0.9525 0.9525 0.9525)
 				(span 1 1)
@@
 				)
 			)
-			(table_cell "200K"
+			(table_cell "143K"
 				(exclude_from_sim no)
-				(at 231.14 135.89 0)
-				(size 10.16 2.54)
+				(at 223.52 147.32 0)
+				(size 8.89 2.54)
 				(margins 0.9525 0.9525 0.9525 0.9525)
 				(span 1 1)
@@
 				)
 			)
-			(table_cell "1100KHZ"
+			(table_cell "10.2K"
 				(exclude_from_sim no)
-				(at 220.98 138.43 0)
-				(size 10.16 2.54)
+				(at 232.41 147.32 0)
+				(size 8.89 2.54)
 				(margins 0.9525 0.9525 0.9525 0.9525)
 				(span 1 1)
@@
 				)
 			)
-			(table_cell "90.9K"
+			(table_cell "5V"
 				(exclude_from_sim no)
-				(at 231.14 138.43 0)
-				(size 10.16 2.54)
+				(at 215.9 149.86 0)
+				(size 7.62 2.54)
 				(margins 0.9525 0.9525 0.9525 0.9525)
 				(span 1 1)
@@
 				)
 			)
-		)
-	)
-	(table
-		(column_count 3)
-		(border
-			(external yes)
-			(header yes)
-			(stroke
-				(width 0)
-				(type solid)
-			)
-		)
-		(separators
-			(rows yes)
-			(cols yes)
-			(stroke
-				(width 0)
-				(type solid)
-			)
-		)
-		(column_widths 7.62 8.89 8.89)
-		(row_heights 2.54 2.54 2.54 2.54)
-		(cells
-			(table_cell "Vout"
+			(table_cell "53.6K"
 				(exclude_from_sim no)
-				(at 215.9 142.24 0)
-				(size 7.62 2.54)
+				(at 223.52 149.86 0)
+				(size 8.89 2.54)
 				(margins 0.9525 0.9525 0.9525 0.9525)
 				(span 1 1)
@@
 				)
 			)
-			(table_cell "R_上"
+			(table_cell "10.2K"
 				(exclude_from_sim no)
-				(at 223.52 142.24 0)
+				(at 232.41 149.86 0)
 				(size 8.89 2.54)
 				(margins 0.9525 0.9525 0.9525 0.9525)
@@
 				)
 			)
-			(table_cell "R_下"
+		)
+	)
+	(table
+		(column_count 2)
+		(border
+			(external yes)
+			(header yes)
+			(stroke
+				(width 0)
+				(type solid)
+			)
+		)
+		(separators
+			(rows yes)
+			(cols yes)
+			(stroke
+				(width 0)
+				(type solid)
+			)
+		)
+		(column_widths 10.16 10.16)
+		(row_heights 2.54 2.54 2.54 2.54 2.54)
+		(cells
+			(table_cell "Fsw"
 				(exclude_from_sim no)
-				(at 232.41 142.24 0)
-				(size 8.89 2.54)
+				(at 220.98 128.27 0)
+				(size 10.16 2.54)
 				(margins 0.9525 0.9525 0.9525 0.9525)
 				(span 1 1)
@@
 				)
 			)
-			(table_cell "3.3V"
+			(table_cell "R"
 				(exclude_from_sim no)
-				(at 215.9 144.78 0)
-				(size 7.62 2.54)
+				(at 231.14 128.27 0)
+				(size 10.16 2.54)
 				(margins 0.9525 0.9525 0.9525 0.9525)
 				(span 1 1)
@@
 				)
 			)
-			(table_cell "31.6K"
+			(table_cell "200KHz"
 				(exclude_from_sim no)
-				(at 223.52 144.78 0)
-				(size 8.89 2.54)
+				(at 220.98 130.81 0)
+				(size 10.16 2.54)
 				(margins 0.9525 0.9525 0.9525 0.9525)
 				(span 1 1)
@@
 				)
 			)
-			(table_cell "10.2K"
+			(table_cell "500K"
 				(exclude_from_sim no)
-				(at 232.41 144.78 0)
-				(size 8.89 2.54)
+				(at 231.14 130.81 0)
+				(size 10.16 2.54)
 				(margins 0.9525 0.9525 0.9525 0.9525)
 				(span 1 1)
@@
 				)
 			)
-			(table_cell "12V"
+			(table_cell "330KHz"
 				(exclude_from_sim no)
-				(at 215.9 147.32 0)
-				(size 7.62 2.54)
+				(at 220.98 133.35 0)
+				(size 10.16 2.54)
 				(margins 0.9525 0.9525 0.9525 0.9525)
 				(span 1 1)
@@
 				)
 			)
-			(table_cell "143K"
+			(table_cell "301K"
 				(exclude_from_sim no)
-				(at 223.52 147.32 0)
-				(size 8.89 2.54)
+				(at 231.14 133.35 0)
+				(size 10.16 2.54)
 				(margins 0.9525 0.9525 0.9525 0.9525)
 				(span 1 1)
@@
 				)
 			)
-			(table_cell "10.2K"
+			(table_cell "500KHz"
 				(exclude_from_sim no)
-				(at 232.41 147.32 0)
-				(size 8.89 2.54)
+				(at 220.98 135.89 0)
+				(size 10.16 2.54)
 				(margins 0.9525 0.9525 0.9525 0.9525)
 				(span 1 1)
@@
 				)
 			)
-			(table_cell "5V"
+			(table_cell "200K"
 				(exclude_from_sim no)
-				(at 215.9 149.86 0)
-				(size 7.62 2.54)
+				(at 231.14 135.89 0)
+				(size 10.16 2.54)
 				(margins 0.9525 0.9525 0.9525 0.9525)
 				(span 1 1)
@@
 				)
 			)
-			(table_cell "53.6K"
+			(table_cell "1100KHZ"
 				(exclude_from_sim no)
-				(at 223.52 149.86 0)
-				(size 8.89 2.54)
+				(at 220.98 138.43 0)
+				(size 10.16 2.54)
 				(margins 0.9525 0.9525 0.9525 0.9525)
 				(span 1 1)
@@
 				)
 			)
-			(table_cell "10.2K"
+			(table_cell "90.9K"
 				(exclude_from_sim no)
-				(at 232.41 149.86 0)
-				(size 8.89 2.54)
+				(at 231.14 138.43 0)
+				(size 10.16 2.54)
 				(margins 0.9525 0.9525 0.9525 0.9525)
 				(span 1 1)

Commit message: 布局初步结束
Connections:
- net GND: now also U3.11 (EP)
- no-connect marks 3 -> 2
Changed lines of the file:
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@@
 	)
 	(no_connect
-		(at 130.81 40.64)
-	)
-	(no_connect
 		(at 130.81 53.34)
 	)
@@
 	(wire
 		(pts
+			(xy 130.81 40.64) (xy 132.08 40.64)
+		)
+		(stroke
+			(width 0)
+			(type default)
+		)
+	)
+	(wire
+		(pts
 			(xy 116.84 135.89) (xy 107.95 135.89)
 		)
@@
 	)
 	(table
-		(column_count 3)
+		(column_count 2)
 		(border
 			(external yes)
@@
 			)
 		)
-		(column_widths 7.62 8.89 8.89)
-		(row_heights 2.54 2.54 2.54 2.54)
+		(column_widths 10.16 10.16)
+		(row_heights 2.54 2.54 2.54 2.54 2.54)
 		(cells
-			(table_cell "Vout"
+			(table_cell "Fsw"
 				(exclude_from_sim no)
-				(at 215.9 142.24 0)
-				(size 7.62 2.54)
+				(at 220.98 128.27 0)
+				(size 10.16 2.54)
 				(margins 0.9525 0.9525 0.9525 0.9525)
 				(span 1 1)
@@
 				)
 			)
-			(table_cell "R_上"
+			(table_cell "R"
 				(exclude_from_sim no)
-				(at 223.52 142.24 0)
-				(size 8.89 2.54)
+				(at 231.14 128.27 0)
+				(size 10.16 2.54)
 				(margins 0.9525 0.9525 0.9525 0.9525)
 				(span 1 1)
@@
 				)
 			)
-			(table_cell "R_下"
+			(table_cell "200KHz"
 				(exclude_from_sim no)
-				(at 232.41 142.24 0)
-				(size 8.89 2.54)
+				(at 220.98 130.81 0)
+				(size 10.16 2.54)
 				(margins 0.9525 0.9525 0.9525 0.9525)
 				(span 1 1)
@@
 				)
 			)
-			(table_cell "3.3V"
+			(table_cell "500K"
 				(exclude_from_sim no)
-				(at 215.9 144.78 0)
-				(size 7.62 2.54)
+				(at 231.14 130.81 0)
+				(size 10.16 2.54)
 				(margins 0.9525 0.9525 0.9525 0.9525)
 				(span 1 1)
@@
 				)
 			)
-			(table_cell "31.6K"
+			(table_cell "330KHz"
 				(exclude_from_sim no)
-				(at 223.52 144.78 0)
-				(size 8.89 2.54)
+				(at 220.98 133.35 0)
+				(size 10.16 2.54)
 				(margins 0.9525 0.9525 0.9525 0.9525)
 				(span 1 1)
@@
 				)
 			)
-			(table_cell "10.2K"
+			(table_cell "301K"
 				(exclude_from_sim no)
-				(at 232.41 144.78 0)
-				(size 8.89 2.54)
+				(at 231.14 133.35 0)
+				(size 10.16 2.54)
 				(margins 0.9525 0.9525 0.9525 0.9525)
 				(span 1 1)
@@
 				)
 			)
-			(table_cell "12V"
+			(table_cell "500KHz"
 				(exclude_from_sim no)
-				(at 215.9 147.32 0)
-				(size 7.62 2.54)
+				(at 220.98 135.89 0)
+				(size 10.16 2.54)
 				(margins 0.9525 0.9525 0.9525 0.9525)
 				(span 1 1)
@@
 				)
 			)
-			(table_cell "143K"
+			(table_cell "200K"
 				(exclude_from_sim no)
-				(at 223.52 147.32 0)
-				(size 8.89 2.54)
+				(at 231.14 135.89 0)
+				(size 10.16 2.54)
 				(margins 0.9525 0.9525 0.9525 0.9525)
 				(span 1 1)
@@
 				)
 			)
-			(table_cell "10.2K"
+			(table_cell "1100KHZ"
 				(exclude_from_sim no)
-				(at 232.41 147.32 0)
-				(size 8.89 2.54)
+				(at 220.98 138.43 0)
+				(size 10.16 2.54)
 				(margins 0.9525 0.9525 0.9525 0.9525)
 				(span 1 1)
@@
 				)
 			)
-			(table_cell "5V"
+			(table_cell "90.9K"
 				(exclude_from_sim no)
-				(at 215.9 149.86 0)
-				(size 7.62 2.54)
+				(at 231.14 138.43 0)
+				(size 10.16 2.54)
 				(margins 0.9525 0.9525 0.9525 0.9525)
 				(span 1 1)
@@
 				)
 			)
-			(table_cell "53.6K"
+		)
+	)
+	(table
+		(column_count 3)
+		(border
+			(external yes)
+			(header yes)
+			(stroke
+				(width 0)
+				(type solid)
+			)
+		)
+		(separators
+			(rows yes)
+			(cols yes)
+			(stroke
+				(width 0)
+				(type solid)
+			)
+		)
+		(column_widths 7.62 8.89 8.89)
+		(row_heights 2.54 2.54 2.54 2.54)
+		(cells
+			(table_cell "Vout"
 				(exclude_from_sim no)
-				(at 223.52 149.86 0)
-				(size 8.89 2.54)
+				(at 215.9 142.24 0)
+				(size 7.62 2.54)
 				(margins 0.9525 0.9525 0.9525 0.9525)
 				(span 1 1)
@@
 				)
 			)
-			(table_cell "10.2K"
+			(table_cell "R_上"
 				(exclude_from_sim no)
-				(at 232.41 149.86 0)
+				(at 223.52 142.24 0)
 				(size 8.89 2.54)
 				(margins 0.9525 0.9525 0.9525 0.9525)
@@
 				)
 			)
-		)
-	)
-	(table
-		(column_count 2)
-		(border
-			(external yes)
-			(header yes)
-			(stroke
-				(width 0)
-				(type solid)
-			)
-		)
-		(separators
-			(rows yes)
-			(cols yes)
-			(stroke
-				(width 0)
-				(type solid)
-			)
-		)
-		(column_widths 10.16 10.16)
-		(row_heights 2.54 2.54 2.54 2.54 2.54)
-		(cells
-			(table_cell "Fsw"
+			(table_cell "R_下"
 				(exclude_from_sim no)
-				(at 220.98 128.27 0)
-				(size 10.16 2.54)
+				(at 232.41 142.24 0)
+				(size 8.89 2.54)
 				(margins 0.9525 0.9525 0.9525 0.9525)
 				(span 1 1)
@@
 				)
 			)
-			(table_cell "R"
+			(table_cell "3.3V"
 				(exclude_from_sim no)
-				(at 231.14 128.27 0)
-				(size 10.16 2.54)
+				(at 215.9 144.78 0)
+				(size 7.62 2.54)
 				(margins 0.9525 0.9525 0.9525 0.9525)
 				(span 1 1)
@@
 				)
 			)
-			(table_cell "200KHz"
+			(table_cell "31.6K"
 				(exclude_from_sim no)
-				(at 220.98 130.81 0)
-				(size 10.16 2.54)
+				(at 223.52 144.78 0)
+				(size 8.89 2.54)
 				(margins 0.9525 0.9525 0.9525 0.9525)
 				(span 1 1)
@@
 				)
 			)
-			(table_cell "500K"
+			(table_cell "10.2K"
 				(exclude_from_sim no)
-				(at 231.14 130.81 0)
-				(size 10.16 2.54)
+				(at 232.41 144.78 0)
+				(size 8.89 2.54)
 				(margins 0.9525 0.9525 0.9525 0.9525)
 				(span 1 1)
@@
 				)
 			)
-			(table_cell "330KHz"
+			(table_cell "12V"
 				(exclude_from_sim no)
-				(at 220.98 133.35 0)
-				(size 10.16 2.54)
+				(at 215.9 147.32 0)
+				(size 7.62 2.54)
 				(margins 0.9525 0.9525 0.9525 0.9525)
 				(span 1 1)
@@
 				)
 			)
-			(table_cell "301K"
+			(table_cell "143K"
 				(exclude_from_sim no)
-				(at 231.14 133.35 0)
-				(size 10.16 2.54)
+				(at 223.52 147.32 0)
+				(size 8.89 2.54)
 				(margins 0.9525 0.9525 0.9525 0.9525)
 				(span 1 1)
@@
 				)
 			)
-			(table_cell "500KHz"
+			(table_cell "10.2K"
 				(exclude_from_sim no)
-				(at 220.98 135.89 0)
-				(size 10.16 2.54)
+				(at 232.41 147.32 0)
+				(size 8.89 2.54)
 				(margins 0.9525 0.9525 0.9525 0.9525)
 				(span 1 1)
@@
 				)
 			)
-			(table_cell "200K"
+			(table_cell "5V"
 				(exclude_from_sim no)
-				(at 231.14 135.89 0)
-				(size 10.16 2.54)
+				(at 215.9 149.86 0)
+				(size 7.62 2.54)
 				(margins 0.9525 0.9525 0.9525 0.9525)
 				(span 1 1)
@@
 				)
 			)
-			(table_cell "1100KHZ"
+			(table_cell "53.6K"
 				(exclude_from_sim no)
-				(at 220.98 138.43 0)
-				(size 10.16 2.54)
+				(at 223.52 149.86 0)
+				(size 8.89 2.54)
 				(margins 0.9525 0.9525 0.9525 0.9525)
 				(span 1 1)
@@
 				)
 			)
-			(table_cell "90.9K"
+			(table_cell "10.2K"
 				(exclude_from_sim no)
-				(at 231.14 138.43 0)
-				(size 10.16 2.54)
+				(at 232.41 149.86 0)
+				(size 8.89 2.54)
 				(margins 0.9525 0.9525 0.9525 0.9525)
 				(span 1 1)
@@
 					(unit 1)
 				)
+			)
+		)
+	)
+	(symbol
+		(lib_id "power:GND")
+		(at 132.08 40.64 90)
+		(unit 1)
+		(exclude_from_sim no)
+		(in_bom yes)
+		(on_board yes)
+		(dnp no)
+		(property "Reference" "#PWR066"
+			(at 138.43 40.64 0)
+			(effects
+				(font
+					(size 1.27 1.27)
+				)
+				(hide yes)
+			)
+		)
+		(property "Value" "GND"
+			(at 134.62 37.338 0)
+			(effects
+				(font
+					(size 1.27 1.27)
+				)
+				(hide yes)
+			)
+		)
+		(property "Footprint" ""
+			(at 132.08 40.64 0)
+			(effects
+				(font
+					(size 1.27 1.27)
+				)
+				(hide yes)
+			)
+		)
+		(property "Datasheet" ""
+			(at 132.08 40.64 0)
+			(effects
+				(font
+					(size 1.27 1.27)
+				)
+				(hide yes)
+			)
+		)
+		(property "Description" "Power symbol creates a global label with name \"GND\" , ground"
+			(at 132.08 40.64 0)
+			(effects
+				(font
+					(size 1.27 1.27)
+				)
+				(hide yes)
+			)
+		)
+		(pin "1"
+		)
+		(instances
+			(project "DriverBoard"
+				(path "/6b2aea6d-5084-4a15-abee-69a455b7078c/ecd3cbd5-4e2a-4cbd-93e4-e6de56463e65"
+					(reference "#PWR066")
+					(unit 1)
+				)
